File: KiCAD/ArEG/ArEG.kicad_pcb (KiCad board)
At the start: 2 copper layers, 67 parts, among them J1 GATE_ACTIVE, J2 ERK_PWR, J3 Gate_Thru, J4 Gate_In, J5 ArduinoISP, J6 DELAYED_GATE, J7 INV_OUT, J8 OUT, Q1 2SA1015, SW1 Manual_Gate, SW2 Speed, U1 ATmega328-PU, U2 TL072, U3 TL072, Y1 16MHz

Commit message: Panel design
Parts:
- removed C11: 0.1u, Capacitor_THT:C_Disc_D3.0mm_W1.6mm_P2.50mm
- removed C8: 1u, Capacitor_THT:C_Disc_D4.3mm_W1.9mm_P5.00mm
- removed R10: 1k, Resistor_THT:R_Axial_DIN0207_L6.3mm_D2.5mm_P10.16mm_Horizontal
- added G***: LOGO, myfootprint:Silk_PNPN_Thyristor_1200dpi, F.Cu at (132.7, 126.4)
- added G***: LOGO, myfootprint:Silk_PNPN_Manufactory_600dpi, F.Cu at (122.6, 125.1)
- added H1: MountingHole, MountingHole:MountingHole_3.2mm_M3, F.Cu at (101.6, 48.3)
- added H2: MountingHole, MountingHole:MountingHole_3.2mm_M3, F.Cu at (101.6, 139.7)
- added H3: MountingHole, MountingHole:MountingHole_3.2mm_M3, F.Cu at (162.6, 48.3)
- added H4: MountingHole, MountingHole:MountingHole_3.2mm_M3, F.Cu at (163.8, 139.7)
- added TP1: TP_Threshold, TestPoint:TestPoint_Pad_D1.0mm, F.Cu at (139.7, 88.9)
- added TP2: TP_ADSR, TestPoint:TestPoint_Pad_D1.0mm, F.Cu at (151.1, 108.0)
- added TP3: TP_DelayTime, TestPoint:TestPoint_Pad_D1.0mm, F.Cu at (152.4, 63.5)
- J3: value Gate_Thru -> GATE_IN; footprint Connector_JST:JST_XH_B2B-XH-A_1x02_P2.50mm_Vertical -> Connector_JST:JST_XH_B3B-XH-A_1x03_P2.50mm_Vertical
- J4: value Gate_In -> OUTPUT; footprint Connector_JST:JST_XH_B2B-XH-A_1x02_P2.50mm_Vertical -> Connector_JST:JST_XH_B3B-XH-A_1x03_P2.50mm_Vertical
- J7: value INV_OUT -> TP_GND; footprint Connector_JST:JST_XH_B2B-XH-A_1x02_P2.50mm_Vertical -> Connector_PinHeader_2.54mm:PinHeader_1x02_P2.54mm_Vertical
- J8: value OUT -> TP_GND; footprint Connector_JST:JST_XH_B2B-XH-A_1x02_P2.50mm_Vertical -> Connector_PinHeader_2.54mm:PinHeader_1x02_P2.54mm_Vertical
- R23: value 4.7k -> 1k
- R9: value 1k -> 33
- SW1: value Manual_Gate -> MANUAL_GATE
- U1: footprint Package_DIP:DIP-28_W7.62mm_LongPads -> Package_DIP:DIP-28_W7.62mm_Socket_LongPads
- U2: value TL072 -> NJM2904; footprint Package_DIP:DIP-8_W7.62mm_LongPads -> Package_DIP:DIP-8_W7.62mm_Socket_LongPads
- U3: footprint Package_DIP:DIP-8_W7.62mm_LongPads -> Package_DIP:DIP-8_W7.62mm_Socket_LongPads
- moved J6 97.8 mm to (105.4, 100.3), turned to 90 degrees
- moved D4 89.8 mm to (158.8, 57.8), turned to 90 degrees
- moved SW1 81.2 mm to (105.4, 111.1), turned to 90 degrees
- moved J7 78.8 mm to (104.1, 127.0), turned to 90 degrees
- moved J8 75.0 mm to (152.4, 50.8)
- moved J1 72.5 mm to (104.1, 67.3)
- moved D6 71.2 mm to (158.8, 68.6), turned to 90 degrees
- moved R7 69.2 mm to (122.6, 117.5), turned to 180 degrees
- moved J3 66.0 mm to (118.1, 137.2), turned to 180 degrees
- moved C2 63.8 mm to (120.7, 66.0)
- moved R18 63.6 mm to (165.7, 55.9), turned to 270 degrees
- moved C9 54.6 mm to (147.3, 90.2), turned to 180 degrees
- moved RV1 54.4 mm to (170.2, 137.2)
- moved D1 53.9 mm to (119.4, 57.1)
- moved Q1 52.5 mm to (162.6, 81.3), turned to 270 degrees
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Connections:
- C9 pad 1: +12V -> +5V
- J3 pad 2: GND -> Net-(J3-Pad1)
- J4 pad 1: Net-(J3-Pad1) -> /ADSR/ADSR_OUT
- J4 pad 2: GND -> /ADSR/INV_OUT
- J7 pad 1: Net-(J7-Pad1) -> GND
- J8 pad 1: Net-(J8-Pad1) -> GND
- R16 pad 1: Net-(J7-Pad1) -> /ADSR/INV_OUT
- R19 pad 1: Net-(J8-Pad1) -> /ADSR/ADSR_OUT
- RV1 pad 2: Net-(R10-Pad2) -> Delay_Time
- U2 pad 1: Net-(R17-Pad2) -> Threshold
- U2 pad 2: Net-(R20-Pad2) -> Net-(RV3-Pad1)
- U2 pad 3: Net-(RV3-Pad1) -> Net-(R11-Pad2)
- U2 pad 4: -12V -> GND
- U2 pad 5: Net-(R11-Pad2) -> Net-(RV3-Pad1)
- U2 pad 6: Net-(RV3-Pad1) -> Net-(R23-Pad1)
- U2 pad 7: Threshold -> Net-(R23-Pad1)
- U2 pad 8: +12V -> +5V
- U3 pad 5: Net-(R17-Pad2) -> Net-(RV3-Pad1)
- U3 pad 6: Net-(R23-Pad1) -> Net-(R20-Pad2)
- U3 pad 7: Net-(R23-Pad1) -> Net-(R17-Pad2)
Routing:
- net +5V: track 0.00 -> 256.8 mm
- net Net-(RV3-Pad1): track 0.00 -> 152.3 mm
- net Delay_Time: track 0.00 -> 118.1 mm
- net -12V: track 0.00 -> 109.0 mm
- net Gate_Com: track 0.00 -> 94.7 mm
- net +12V: track 0.00 -> 85.5 mm
- net Net-(J6-Pad1): track 0.00 -> 50.0 mm
- net Threshold: track 0.00 -> 39.6 mm
- net Release: track 0.00 -> 39.0 mm
- net Decay: track 0.00 -> 38.4 mm
- net Net-(R17-Pad2): track 0.00 -> 38.4 mm
- net /ADSR/ADSR_OUT: track 0.00 -> 36.8 mm
- net Attack: track 0.00 -> 33.3 mm
- net /ADSR/INV_OUT: track 0.00 -> 31.3 mm
- net Net-(J3-Pad1): track 0.00 -> 26.7 mm
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- added copper zone on B.Cu, net GND
- added copper zone on F.Cu, net GND
Other:
- board outline added: 74.9 x 96.5 mm
- board text added: "+5V"
- board text added: "3 C 2 1"
- board text added: "ADSR"
- board text added: "ARDUINO_ISP"
- board text added: "ATTACK"
- board text added: "ArEG"
- board text added: "DECAY"
- board text added: "DELAY TIME"
- board text added: "DELAYED_GATE"
- board text added: "G"
- board text added: "G ADSR_LED"
- board text added: "G DELAY_LED"
- board text added: "G GATE_LED"
- board text added: "G INV ADSR"
- board text added: "G THRU IN"
- board text added: "GATE_COM"
- board text added: "GATE_IN"
- board text added: "GND"
- board text added: "MANUAL_GATE"
- board text added: "OUT"
- board text added: "RELEASE"
- board text added: "RST"
- board text added: "RXD"
- board text added: "SPEED"
- board text added: "SUSTAIN"
- board text added: "THRESHOLD"
- board text added: "TXD"
- board text added: "Ver.1.0"
- board text added: "https://dad8893.blogspot.com/"
