File: KiCAD/ArEG/ArEG.sch (KiCad schematic (older format))
At the start: 31 parts

Commit message: 入出力端子をまとめる前
Parts:
- removed C? (x2): 22p, symbol Device:C
- removed RV?: 50k, symbol Device:R_POT_TRIM
- removed Y?: 16MHz, symbol Device:Crystal
- added C5: 0.1u, Capacitor_THT:C_Disc_D3.0mm_W1.6mm_P2.50mm, symbol Device:C
- added C6, C7: 22p, Capacitor_THT:C_Disc_D4.3mm_W1.9mm_P5.00mm, symbol Device:C
- added C8: 1u, Capacitor_THT:C_Disc_D4.3mm_W1.9mm_P5.00mm, symbol Device:C
- added D6: YELLOW, Connector_JST:JST_XH_B2B-XH-A_1x02_P2.50mm_Vertical, symbol Device:LED
- added J5: ArduinoISP, Connector_PinHeader_2.54mm:PinHeader_1x04_P2.54mm_Vertical, symbol Connector_Generic:Conn_01x04
- added R10, R5: 1k, Resistor_THT:R_Axial_DIN0207_L6.3mm_D2.5mm_P10.16mm_Horizontal, symbol Device:R
- added Y1: 16MHz, Crystal:Crystal_HC18-U_Vertical, symbol Device:Crystal
- C1, C3: renamed from C?; footprint (none) -> Capacitor_THT:CP_Radial_D5.0mm_P2.50mm
- C2: renamed from C?; footprint (none) -> Capacitor_THT:CP_Radial_D6.3mm_P2.50mm
- C4: renamed from C?; footprint (none) -> Capacitor_THT:C_Disc_D3.0mm_W1.6mm_P2.50mm
- D1, D2, D3: renamed from D?; footprint (none) -> LED_THT:LED_D3.0mm
- D4: renamed from D?; footprint (none) -> Connector_JST:JST_XH_B2B-XH-A_1x02_P2.50mm_Vertical
- D5, D7, D8: renamed from D?; footprint (none) -> Diode_THT:D_DO-34_SOD68_P7.62mm_Horizontal
- J1: renamed from J?; footprint (none) -> Connector_PinHeader_2.54mm:PinHeader_1x02_P2.54mm_Vertical
- J2: renamed from J?; footprint (none) -> Connector_IDC:IDC-Header_2x08_P2.54mm_Vertical
- J3, J4, J6: renamed from J?; footprint (none) -> Connector_JST:JST_XH_B2B-XH-A_1x02_P2.50mm_Vertical
- R1, R2, R3, R4, R6, R8, R9: renamed from R?; footprint (none) -> Resistor_THT:R_Axial_DIN0207_L6.3mm_D2.5mm_P10.16mm_Horizontal
- R7: renamed from R?; value 100k -> Open; footprint (none) -> Resistor_THT:R_Axial_DIN0207_L6.3mm_D2.5mm_P10.16mm_Horizontal
- RV1: renamed from RV?; footprint (none) -> Potentiometer_THT:Potentiometer_Alps_RK09Y11_Single_Horizontal
- SW1: renamed from SW?; footprint (none) -> Connector_JST:JST_XH_B2B-XH-A_1x02_P2.50mm_Vertical
- U1: renamed from U?; footprint Package_DIP:DIP-28_W7.62mm -> Package_DIP:DIP-28_W7.62mm_LongPads
Connections:
- net Delay_Time: now also U1.23 (PC0), C8.2, R10.1; no longer RV1.2, U1.25 (PC2)
- net Delayed_Gate: now also U1.6 (PD4); no longer U1.4 (PD2)
- net GND: now also C5.1, C6.1, C7.2, C8.1, D6.1 (K), J5.4 (Pin_4)
- net Threshold: now also U1.4 (PD2); no longer U1.23 (PC0)
- net at U1.9 (XTAL1/PB6): now also C6.2, Y1.1
- net at U1.10 (XTAL2/PB7): now also C7.1, Y1.2
- net RST: now reaches U1.1 (~RESET~/PC6)
- net RST: now also J5.1 (Pin_1)
- net Delayed_LED: now reaches U1.18 (PB4)
- net Delayed_LED: now also R5.2
- net RXD: now reaches U1.2 (PD0)
- net RXD: now also J5.2 (Pin_2)
- net at U1.21 (AREF): now also C5.2
- net TXD: now reaches U1.3 (PD1)
- net TXD: now also J5.3 (Pin_3)
- net Sustain renamed Decay
- net Threshold_Level: no longer names the net of U1.24 (PC1)
- new net: R10.2, RV1.2
- new net: D6.2 (A), R5.1
- no-connect marks 15 -> 11
Other:
- note added: "A0"
- note added: "D0\nD1\nD2\nD3\nD4\nD5\nD6\nD7"
- note added: "D12\nD13"
- moved on the sheet: C4, D4, D5, D7, D8, J3, J4, J6, R4, R6, R7, R8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

Commit message: Panel design
Parts:
- removed C8: 1u, Capacitor_THT:C_Disc_D4.3mm_W1.9mm_P5.00mm, symbol Device:C
- removed J3: Gate_Thru, Connector_JST:JST_XH_B2B-XH-A_1x02_P2.50mm_Vertical, symbol Connector_Generic:Conn_01x02
- removed J4: Gate_In, Connector_JST:JST_XH_B2B-XH-A_1x02_P2.50mm_Vertical, symbol Connector_Generic:Conn_01x02
- removed R10: 1k, Resistor_THT:R_Axial_DIN0207_L6.3mm_D2.5mm_P10.16mm_Horizontal, symbol Device:R
- added H1, H2, H3, H4: MountingHole, MountingHole:MountingHole_3.2mm_M3, symbol Mechanical:MountingHole
- added J3: GATE_IN, Connector_JST:JST_XH_B3B-XH-A_1x03_P2.50mm_Vertical, symbol Connector_Generic:Conn_01x03
- added J4: OUTPUT, Connector_JST:JST_XH_B3B-XH-A_1x03_P2.50mm_Vertical, symbol Connector_Generic:Conn_01x03
- added J7, J8: TP_GND, Connector_PinHeader_2.54mm:PinHeader_1x02_P2.54mm_Vertical, symbol Connector_Generic:Conn_01x02
- added TP3: TP_DelayTime, TestPoint:TestPoint_Pad_D1.0mm, symbol Connector:TestPoint
- R9: value 1k -> 33
- SW1: value Manual_Gate -> MANUAL_GATE
- U1: footprint Package_DIP:DIP-28_W7.62mm_LongPads -> Package_DIP:DIP-28_W7.62mm_Socket_LongPads
Connections:
- net Delay_Time: now also RV1.2, TP3.1
- net GND: now also J3.3 (Pin_3), J4.3 (Pin_3), J7.1 (Pin_1), J7.2 (Pin_2), J8.1 (Pin_1), J8.2 (Pin_2)
- net at R6.1, R7.2: now also J3.1 (Pin_1), J3.2 (Pin_2)
- new net ADSR/ADSR_OUT: J4.1 (Pin_1)
- new net ADSR/INV_OUT: J4.2 (Pin_2)
Other:
- note added: "ADSR_OUT\nINV_OUT\nGND"
- note added: "IN\nTHRU\nGND"
- moved on the sheet: D4, D6, R4, R5, R8, R9, SW1
